File: kicad/MiniPicoPCB.kicad_pcb (KiCad board)
At the start: 2 copper layers, 58 x 74 mm, 15 parts, among them J1 Screw_Terminal_01x05, J10 Screw_Terminal_01x05, J11 Conn_01x20_Socket, J12 Conn_01x20_Socket, J2 Screw_Terminal_01x05, J3 Screw_Terminal_01x05, J4 Screw_Terminal_01x05, J5 Screw_Terminal_01x05, J6 Screw_Terminal_01x05, J7 Screw_Terminal_01x05, J8 Screw_Terminal_01x05, J9 Screw_Terminal_01x05

Commit message: Update schematic, PCB, assets
Other:
- outline, holes or cut-outs redrawn
- board text added: "${PCB_VERSION}"
- board text added: "aisler.net (2026-09-21)"
- board text removed: "aisler.net (2026-07-22)"

Commit message: Update footprint warning
Other:
- board text added: "aisler.net (2026-10-XX)"
- board text removed: "aisler.net (2026-09-21)"
Changed lines of the file:
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@@
 	(title_block
 		(title "${TITLE_NAME}")
-		(date "2026-09-21")
+		(date "2026-10-06")
 		(rev "${PCB_VERSION}")
 		(comment 2 "${PROJECT_LINK}")
@@
 		)
 	)
-	(gr_text "aisler.net (2026-09-21)"
+	(gr_text "aisler.net (2026-10-XX)"
 		(locked yes)
 		(at 142.494 88.646 90)
@@
 		)
 	)
-	(group ""
-		(locked yes)
-		(members "26e591b4-5c1a-4491-b443-91aa5136db5e" "9ae88b0e-dabc-45ce-aa9b-188e970a2ce0"
-			"ede8d774-c38b-44b7-ba61-d4935b1c3be3" "f009d545-2ba7-43dd-90d1-ca531fc30351"
-		)
-	)
-	(group ""
-		(locked yes)
-		(members "1819a438-b6c7-4f8d-ab9f-64195fe002a8" "52113f6c-a95c-4011-9135-de9f1fd213bb"
-			"62e23296-3fcb-404c-8f10-d4ccbd7a1da1" "a7342972-fa2e-4752-bb42-62e09b4058c9"
-		)
-	)
